File: HackerBadgePCBV3 (Simplified).kicad_sch (KiCad schematic)
At the start: 14 parts

Commit message: Tweaks
Connections:
- net at R2.2: no longer D3.2 (A)
- net at D2.2 (A): now also R5.2; no longer R1.2
- net at R3.2: no longer D4.2 (A)
- net at D5.2 (A): no longer R5.2
- net at R4.2: no longer D1.2 (A)
Other:
- moved on the sheet: D1, D2, D3, D4, D5, D6, R1, R2, R3

Commit message: Further tweaks
Connections:
- net at R2.2: now also D5.2 (A)
- net at R3.2: now also D3.2 (A)
- net at R4.2: now also D4.2 (A)
- net at D1.2 (A): now also R1.2
Other:
- moved on the sheet: D1, D2, D3, D4, D5, D6, R1, R2, R3, R4, R5, R6
