File: keyboard.kicad_sch (KiCad schematic)
At the start: 110 parts, among them IC1 STM32F072C8T6, IC2 REG1117, IC3 741G08DBV, SW1 324_SW324_SWITCH_FOOT_HOLE, SW10 KAILH_SWITCH_SOCKET_KAILH_SWI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, SW11 KAILH_SWITCH_SOCKET_KAILH_SWI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, SW12 KAILH_SWITCH_SOCKET_KAILH_SWI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, SW13 KAILH_SWITCH_SOCKET_KAILH_SWI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, SW14 KAILH_SWITCH_SOCKET_KAILH_SWI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, SW15 KAILH_SWITCH_SOCKET_KAILH_SWI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

Commit message: Add files via upload
Parts:
- added TF1: TF-CARD H1.8, easyeda2kicad:TF-SMD_TF-CARD-H1.8, symbol easyeda2kicad:TF-CARDH1.8
- IC3: LCSC Part (none) -> C434068
- JP1: LCSC Part (none) -> C7470081
- LED1, LED10, LED11, LED12, LED13, LED14, LED15, LED2, LED3, LED4, LED5, LED6, LED7, LED8, LED9: LCSC Part (none) -> C4154882
- SD1: LCSC Part (none) -> C7529389
Connections:
- net at LED5.DIN (DI): now also LED6.DOUT (DO); no longer LED4.DOUT (DO)
- net at LED5.DOUT (DO): now also LED4.DIN (DI); no longer LED6.DIN (DI)
- net at LED10.DIN (DI): now also LED11.DOUT (DO); no longer LED7.DOUT (DO)
- net at LED10.DOUT (DO): now also LED9.DOUT (DO); no longer LED11.DIN (DI)
- net at LED8.DIN (DI): now also LED7.DOUT (DO); no longer LED9.DOUT (DO)
- net at LED8.DOUT (DO): now also LED9.DIN (DI); no longer LED7.DIN (DI)
- net at LED1.DOUT (DO): now also LED4.DOUT (DO); no longer LED4.DIN (DI)
- net at LED12.DIN (DI): now also LED15.DIN (DI); no longer LED11.DOUT (DO)
- net at LED12.DOUT (DO): now also LED11.DIN (DI); no longer LED15.DIN (DI)
- new net: LED6.DIN (DI), LED7.DIN (DI)
- no-connect marks 0 -> 1
